File: hardware/eda/UFH-CPU/valhalla-ufh-cpu-SMT.kicad_pcb (KiCad board)
At the start: 2 copper layers, 90.9 x 84.6 mm, 70 parts, among them J1 TerminalBlock, 5.08, J2 TerminalBlock, 5.08, J3 TerminalBlock, 5.08, J4 MaleHeader, 2.54, shrouded, J5 TerminalBlock, 5.08, J6 TerminalBlock, 5.08, Q1 MMBT4403, Q2 PN2222A, U1 6N137, U10 74LVC2G125, U11 MAX3483, U12 ISO1410, U2 6N137, U3 6N137, U4 6N137, U5 6N137, U6 74LS123, U7 ATmega328PB-A, U8 74HC595, Y1 7.3728 MHz

Commit message: UPDATE: UFH CPU board layout complete
Parts:
- added REF**: OSHW-Logo2_14.6x12mm_SilkScreen, Symbol:OSHW-Logo2_14.6x12mm_SilkScreen, F.Cu at (194.6, 105.7)
- renumbered C2 to C1, C11 to C10, C9 to C11, C1 to C2, C4 to C3, C3 to C4, C10 to C9, D13 to D1, D5 to D10, D6 to D11, D3 to D13, D1 to D2, D2 to D3, D7 to D5, D8 to D6, D9 to D7, D10 to D8, D11 to D9, PS2 to PS1, Q2 to Q1, Q1 to Q2, R20 to R1, R15 to R11, R16 to R12, R17 to R13, R1 to R2, R18 to R3, R19 to R4, R2 to R5, R4 to R6, R5 to R7, RL2 to RL12, R7 to RL13, R3 to RL2, R6 to RL3, RL1 to RL4, R11 to RL6, R12 to RL7, R13 to RL8, R14 to RL9, U11 to U10, U12 to U11, U10 to U9
Routing:
- net Net-(U6A-RCext): track 7.76 -> 11.5 mm
- net /~{PUMP_STBY}: track 35.8 -> 32.3 mm, vias 3 -> 1
- net Net-(U10-DI): track 102.6 -> 102.1 mm
- net /PWM_REQ: track 45.2 -> 45.7 mm
- net /~{PUMP_LVWR}: track 37.8 -> 38.3 mm
Other:
- board text added: "20240213"
- board text added: "A"
- board text added: "ACK"
- board text added: "B"
- board text added: "BOTC"
- board text added: "GND"
- board text added: "H+"
- board text added: "H-"
- board text added: "Heat"
- board text added: "ICSP"
- board text added: "Interlock"
- board text added: "L"
- board text added: "MAINS"
- board text added: "Modbus"
- board text added: "N"
- board text added: "PWM"
- board text added: "REQ"
- board text added: "TOPC"
- board text added: "TOPS"
- board text added: "Underfloor Heating CPU"
- board text added: "VBUS"
- board text added: "VCC"
- board text added: "~{ACK}"
- board text added: "~{REQ}"
