File: hardware/eda/UFH-CPU/valhalla-ufh-cpu-SMT.kicad_sch (KiCad schematic)
At the start: 69 parts, among them J1 TerminalBlock, 5.08, J2 TerminalBlock, 5.08, J3 TerminalBlock, 5.08, J4 MaleHeader, 2.54, shrouded, J5 TerminalBlock, 5.08, J6 TerminalBlock, 5.08, Q1 MMBT4403, Q2 PN2222A, U1 6N137, U10 74LVC2G125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

Commit message: UPDATE: UFH CPU board layout complete
Parts:
- renumbered C2 to C1, C11 to C10, C9 to C11, C1 to C2, C4 to C3, C3 to C4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
