File: hardware/eda/VLM-CP1/valhalla-MOD-_BUFFER-POWER-active-high.kicad_sch (KiCad schematic)
At the start: 1 part, among them U2 74LS06

Commit message: UPDATE: CPU module trace routing complete
 - remaining stuff: crystal dress-up and silkscreen finish-up
 - we may choose not to get artsy on this one (teardrops and curves) due
   to DRC/real estate constraints.
Parts:
- U2: footprint Package_DIP:DIP-14_W7.62mm_LongPads -> Package_DIP:DIP-14_W7.62mm
Changed lines of the file:
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@@
 			)
 		)
-		(property "Footprint" "Package_DIP:DIP-14_W7.62mm_LongPads"
+		(property "Footprint" "Package_DIP:DIP-14_W7.62mm"
 			(at 127 83.82 0)
 			(effects
