File: hardware/eda/VLM-CP1/valhalla-MOD-_LED-active-high.sch.kicad_sch (KiCad schematic)
At the start: 3 parts, among them U2 74LS06

Commit message: UPDATE: formal dimensions for Valhalla MOD and progrss on CPU
 - added formal dimensions to the Valhalla MOD PSU PCB, to serve as a
   future template and as documentation
 - changed Zener/Schottky symbols to filled variant on same module,
   as customary in the EU
 - solved the Vio independence issue for the UI LEDs on the CPU module
   with a switchable regulator
 - finalized canonical dimensions of the CPU module and placed UI
   LEDs in two rows.
Parts:
- R3: footprint Resistor_THT:R_Axial_DIN0309_L9.0mm_D3.2mm_P12.70mm_Horizontal -> Resistor_THT:R_Axial_DIN0207_L6.3mm_D2.5mm_P10.16mm_Horizontal
Changed lines of the file:
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@@
 			)
 		)
-		(property "Footprint" "Resistor_THT:R_Axial_DIN0309_L9.0mm_D3.2mm_P12.70mm_Horizontal"
+		(property "Footprint" "Resistor_THT:R_Axial_DIN0207_L6.3mm_D2.5mm_P10.16mm_Horizontal"
 			(at 65.532 53.34 90)
 			(effects

Commit message: UPDATE: progress on component placement for CPU module
Parts:
- R3: footprint Resistor_THT:R_Axial_DIN0207_L6.3mm_D2.5mm_P10.16mm_Horizontal -> Resistor_THT:R_Axial_DIN0207_L6.3mm_D2.5mm_P5.08mm_Vertical
Changed lines of the file:
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@@
 			)
 		)
-		(property "Footprint" "Resistor_THT:R_Axial_DIN0207_L6.3mm_D2.5mm_P10.16mm_Horizontal"
+		(property "Footprint" "Resistor_THT:R_Axial_DIN0207_L6.3mm_D2.5mm_P5.08mm_Vertical"
 			(at 65.532 53.34 90)
 			(effects

Commit message: UPDATE: CPU module trace routing complete
 - remaining stuff: crystal dress-up and silkscreen finish-up
 - we may choose not to get artsy on this one (teardrops and curves) due
   to DRC/real estate constraints.
Parts:
- U2: footprint Package_DIP:DIP-14_W7.62mm_LongPads -> Package_DIP:DIP-14_W7.62mm
Changed lines of the file:
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@@
 			)
 		)
-		(property "Footprint" "Package_DIP:DIP-14_W7.62mm_LongPads"
+		(property "Footprint" "Package_DIP:DIP-14_W7.62mm"
 			(at 58.42 68.58 0)
 			(effects
