File: hardware/eda/VLM-_TP/valhalla-MOD-_TEMPLATE.kicad_pcb (KiCad board)
At the start: 2 copper layers, 76.2 x 50.8 mm, 5 parts, among them J1 BUS

Commit message: UPDATE: updated the MOD template to match the latest specification.
Connections:
- J1 pad 12: unconnected-(J1-Pin_12-Pad12) -> /BVCC
- J1 pad 16: unconnected-(J1-Pin_16-Pad16) -> /LVCC
- J1 pad 6: unconnected-(J1-Pin_6-Pad6) -> /DGND
