File: hardware/eda/VLM-XVG/valhalla-MOD-XVR_4IO.kicad_pcb (KiCad board)
At the start: 2 copper layers, 206.2 x 99.6 mm, 131 parts, among them J1 POWER, J14 GLM_F, J15 GLM_F, J16 GLM_F, J17 GLM_F, J18 GLM_B, J19 GLM_B, J2 FIELD, J20 GLM_B, J21 GLM_B, J22 WDM_I, J23 WDM_I, J24 TM, J25 FIM_I, J26 FIM_I, J27 FIM_I, J28 FIM_I, J29 WDM_I, J3 GPIO, J30 FIM_I, J31 TM_0, J32 TM_1, J33 FIM_I, J34 WDM_E, J35 WDM_E, J36 WDM_E, J37 FIM_I, J38 FIM_I, J39 FIM_I, J4 FIM_E, J40 FIM_I, J5 FIM_E, J6 FIM_E, J7 FIM_E, J8 FIM_E, Q1 IRLZ44N, Q2 IRLZ44N, Q3 2N3904, Q4 2N3904, Q5 2N3906, Q6 2N3906, U1 4N35, U2 4N35, U3 74HC14, U4 4N35, U5 4N35, U6 74HC74, U8 74HC123, U9 74HC04

Commit message: UPDATE: MOD-XVR(4IO) done, RTM (panelizing required)
 - fixed silkscreen overhanging the board edge on mainboard
 - ran DRC and fixed or approved all issues
 - we're done here, RTM
  - splitting by sub-pcb and generating Gerbers separately will be done
    on order day (especially since needed sub-pcb quantity differs from
    one).
Parts:
- added ?: , clipboard:e22e6323-0751-47ca-9aea-44c61c1ed047, F.Cu at (121.9, 49.8)
- added ?: , clipboard:e22e6323-0751-47ca-9aea-44c61c1ed047, F.Cu at (121.9, 53.8)
Other:
- board text added: "20251226"
- board text removed: "20251218"

Commit message: UPDATE: improved LVCC rail usage on MOD-XVR(4IO)
  - LVCC now powers the LEDs, the buffer driving them is powered by
    DVCC, this avoids transients caused by UI changes to propagage
    on the digital power rail
  - 74HC04 was replaced by 74HC125
  - also added decoupling capacitors to all logic chips that required
    them
  - changed footprint of Timing Module capacitor to reflect mounting
    (horizontal)
  - re-done routing and adjusted silkscreen in affected areas.
Parts:
- removed ? (x2): , clipboard:e22e6323-0751-47ca-9aea-44c61c1ed047
- removed U9: 74HC04, Package_DIP:DIP-14_W7.62mm
- added C6: 100nF, Capacitor_THT:C_Rect_L4.0mm_W2.5mm_P2.50mm, B.Cu at (90.4, 52.8)
- added C7: 100nF, Capacitor_THT:C_Rect_L4.0mm_W2.5mm_P2.50mm, B.Cu at (167.7, 101.6)
- added C8: 100nF, Capacitor_THT:C_Rect_L4.0mm_W2.5mm_P2.50mm, B.Cu at (190.5, 94.5)
- added U7: 74LS125, Package_DIP:DIP-14_W7.62mm, F.Cu at (87.9, 47.8)
- C5: footprint Capacitor_THT:C_Rect_L9.0mm_W2.5mm_P7.50mm_MKT -> Capacitor_THT:CP_Radial_D5.0mm_P2.00mm
- D26: footprint LED_THT:LED_D3.0mm_Horizontal_O1.27mm_Z2.0mm -> LED_THT:LED_D3.0mm_Horizontal_O3.81mm_Z6.0mm
- D27: footprint LED_THT:LED_D3.0mm_Horizontal_O3.81mm_Z6.0mm -> LED_THT:LED_D3.0mm_Horizontal_O1.27mm_Z2.0mm
- F1, F2: value 1AF -> F1A
- moved R31 10.2 mm to (214.4, 92.5), turned to 90 degrees
- moved C5 8.86 mm to (209.3, 92.5), turned to 0 degrees
- moved R35 7.24 mm to (112.2, 36.0)
- moved D28 6.08 mm to (120.1, 39.4)
- moved R32 5.23 mm to (112.2, 45.3)
- moved D25 4.08 mm to (122.7, 44.5)
- moved R33 3.96 mm to (112.2, 42.3)
- moved D27 2.74 mm to (122.7, 39.4)
- moved D26 2.68 mm to (120.1, 44.5)
- moved JP1 2.54 mm to (188.0, 98.2)
- moved R34 1.97 mm to (112.2, 39.0)
Connections:
- D25 pad 1: /DGND -> Net-(D25-K)
- D25 pad 2: Net-(D25-A) -> /LVCC
- D26 pad 1: /DGND -> Net-(D26-K)
- D26 pad 2: Net-(D26-A) -> /LVCC
- D27 pad 1: /DGND -> Net-(D27-K)
- D27 pad 2: Net-(D27-A) -> /LVCC
- D28 pad 1: /DGND -> Net-(D28-K)
- D28 pad 2: Net-(D28-A) -> /LVCC
- R32 pad 2: Net-(D25-A) -> Net-(D25-K)
- R33 pad 2: Net-(D26-A) -> Net-(D26-K)
- R34 pad 2: Net-(D27-A) -> Net-(D27-K)
- R35 pad 2: Net-(D28-A) -> Net-(D28-K)
- U3 pad 10: /ISEC_DGND -> unconnected-(U3-Pad10)
- U3 pad 11: unconnected-(U3-Pad11) -> /ISEC_DGND
Routing:
- net /LVCC: track 68.1 -> 99.8 mm
- net /~{BGPIO_E_0}: track 106.6 -> 89.9 mm
- net Net-(R32-Pad1): track 45.0 -> 28.6 mm
- net /~{BGPIO_E_2}: track 120.1 -> 105.4 mm
- net Net-(R35-Pad1): track 42.8 -> 31.3 mm
- net Net-(J24-Pin_2): track 18.8 -> 8.20 mm
- net /FVCC: track 92.8 -> 102.1 mm
- net Net-(R33-Pad1): track 30.5 -> 22.2 mm
- net /~{BGPIO_E_1}: track 89.7 -> 97.3 mm
- net Net-(D26-A): track 6.89 -> 0.00 mm
- net Net-(D27-K): track 0.00 -> 6.63 mm
- net Net-(D25-K): track 0.00 -> 6.39 mm
- net Net-(D25-A): track 5.81 -> 0.00 mm
- net Net-(D28-K): track 0.00 -> 4.58 mm
- net Net-(R34-Pad1): track 33.8 -> 37.6 mm
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Other:
- board text added: "20260102"
- board text added: "Timing"
- board text removed: "20251226"
- board text removed: "Timing Module"
