File: hardware/eda/VLM-XVG/valhalla-MOD-XVR_4IO.kicad_sch (KiCad schematic)
At the start: 126 parts, among them J1 POWER, J10 FIM_I, J11 FIM_I, J12 FIM_I, J13 FIM_I, J14 GLM_F, J15 GLM_F, J16 GLM_F, J17 GLM_F, J18 GLM_B, J19 GLM_B, J2 FIELD, J20 GLM_B, J21 GLM_B, J22 WDM_I, J23 WDM_I, J24 TM, J29 WDM_I, J3 GPIO, J31 TM_0, J32 TM_1, J34 WDM_E, J35 WDM_E, J36 WDM_E, J4 FIM_E, J5 FIM_E, J6 FIM_E, J7 FIM_E, J8 FIM_E, J9 FIM_I, Q1 IRLZ44N, Q2 IRLZ44N, Q3 2N3904, Q4 2N3904, Q5 2N3906, Q6 2N3906, U1 4N35, U2 4N35, U3 74HC14, U4 4N35, U5 4N35, U6 74HC74, U8 74HC123, U9 74HC04

Commit message: UPDATE: 1st routing pass done on MOD-XVR(4IO)
 - netclass will have to be re-checked on GPI-Mains
   - clearance/creepage values between the two GPI lines
 - netclass will have to be re-checked on GPO-Power
   - ampacity of entire high-power loop
 - polarization for the field interface modules to be added
   - GPIO line modules are already polarized
   - watchdog/debouncer modules are idempotent
 - silkscreen and mechanical details are last.
Connections:
- net ISEC_DGND: now also U3.10; no longer U3.11
- net ~{BGPIO_E_0}: now also U9.3; no longer U9.9
- net ~{BGPIO_E_1}: now also U9.9; no longer U9.5
- net ~{BGPIO_E_2}: now also U9.1; no longer U9.3
- net ~{BGPIO_E_3}: now also U9.5; no longer U9.1
- net at R32.1: now also U9.4; no longer U9.8
- net at R35.1: now also U9.6; no longer U9.2
- net at R33.1: now also U9.8; no longer U9.6
- net at R34.1: now also U9.2; no longer U9.4
Changed lines of the file:
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@@
 		(lib_id "74xx:74HC04")
 		(at 266.7 187.96 180)
-		(unit 4)
+		(unit 2)
 		(exclude_from_sim no)
 		(in_bom yes)
@@
 				(path "/f06f94c1-3b85-417f-a10f-1ec163aec97d"
 					(reference "U9")
-					(unit 4)
+					(unit 2)
 				)
 			)
@@
 		(lib_id "74xx:74HC04")
 		(at 266.7 201.93 180)
-		(unit 3)
+		(unit 4)
 		(exclude_from_sim no)
 		(in_bom yes)
@@
 				(path "/f06f94c1-3b85-417f-a10f-1ec163aec97d"
 					(reference "U9")
-					(unit 3)
+					(unit 4)
 				)
 			)
@@
 		(lib_id "74xx:74HC14")
 		(at 254 154.94 0)
+		(mirror y)
 		(unit 5)
 		(exclude_from_sim no)
@@
 		(on_board yes)
 		(dnp no)
-		(fields_autoplaced yes)
 		(property "Reference" "U3"
 			(at 254 146.05 0)
@@
 		(lib_id "74xx:74HC04")
 		(at 266.7 215.9 180)
-		(unit 2)
+		(unit 1)
 		(exclude_from_sim no)
 		(in_bom yes)
@@
 				(path "/f06f94c1-3b85-417f-a10f-1ec163aec97d"
 					(reference "U9")
-					(unit 2)
+					(unit 1)
 				)
 			)
@@
 		(lib_id "74xx:74HC04")
 		(at 266.7 229.87 180)
-		(unit 1)
+		(unit 3)
 		(exclude_from_sim no)
 		(in_bom yes)
@@
 				(path "/f06f94c1-3b85-417f-a10f-1ec163aec97d"
 					(reference "U9")
-					(unit 1)
+					(unit 3)
 				)
 			)

Commit message: UPDATE: silkscreen done on mainboard of XVR(4IO)
 - GPIO FIM mechanical polarization also done
Parts:
- removed J10, J11: FIM_I, Connector_PinSocket_2.54mm:PinSocket_1x04_P2.54mm_Vertical, symbol Connector:Conn_01x04_Socket
- removed J12, J13, J9: FIM_I, Connector_PinHeader_2.54mm:PinHeader_1x04_P2.54mm_Vertical, symbol Connector:Conn_01x04_Pin
- added J25, J26, J27, J28, J30, J33: FIM_I, Connector_PinHeader_2.54mm:PinHeader_1x02_P2.54mm_Vertical, symbol Connector:Conn_01x02_Pin
- added J37, J38, J39, J40: FIM_I, Connector_PinSocket_2.54mm:PinSocket_1x02_P2.54mm_Vertical, symbol Connector:Conn_01x02_Socket
Connections:
- net FLED_0: now also J37.2 (Pin_2)
- net FLED_1: now also J38.2 (Pin_2)
- net FLED_2: now also J39.1 (Pin_1)
- net FLED_3: now also J40.1 (Pin_1)
- net ~{FGPIO_I_0}: now also J37.1 (Pin_1)
- net ~{FGPIO_I_1}: now also J38.1 (Pin_1)
- net ~{FGPIO_I_2}: now also J39.2 (Pin_2)
- net ~{FGPIO_I_3}: now also J40.2 (Pin_2)
- net at R6.1: now also J33.1 (Pin_1)
- net at D5.2 (A), D6.1 (K), J6.3 (Pin_3): now also J33.2 (Pin_2)
- net at C1.2, D23.2 (A): now also J27.1 (Pin_1)
- net at D14.2 (-): now also J28.2 (Pin_2)
- net at R5.1: now also J30.1 (Pin_1)
- net at D3.2 (A), D4.1 (K), J6.2 (Pin_2): now also J30.2 (Pin_2)
- net at C2.2, D24.2 (A): now also J28.1 (Pin_1)
- net at D13.2 (-): now also J27.2 (Pin_2)
- net at R17.1: now also J25.2 (Pin_2)
- net at R18.1: now also J26.2 (Pin_2)

Commit message: UPDATE: finished silkscreen on MOD-XVR(4IO)
  - finalized mechanical details of Timing Module interface to
    Watchdog/Debouncer module
  - finalized silkscreen of all daughtercards
  - overhanging parts on main board still need their silkscreen clipped
    to the board edge.
Parts:
- J24: footprint Connector_PinHeader_2.54mm:PinHeader_1x03_P2.54mm_Vertical -> Connector_PinHeader_2.54mm:PinHeader_1x03_P2.54mm_Horizontal
- J31, J32: footprint Connector_PinSocket_2.54mm:PinSocket_1x03_P2.54mm_Vertical -> Connector_PinSocket_2.54mm:PinSocket_1x03_P2.54mm_Horizontal
Connections:
- net WDTM_DGND: now also J24.1 (Pin_1); no longer J24.3 (Pin_3)
- net WDTM_DVCC: now also J24.3 (Pin_3); no longer J24.1 (Pin_1)
Other:
- moved on the sheet: J24
Changed lines of the file:
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@@
 			)
 		)
-		(property "Footprint" "Connector_PinSocket_2.54mm:PinSocket_1x03_P2.54mm_Vertical"
+		(property "Footprint" "Connector_PinSocket_2.54mm:PinSocket_1x03_P2.54mm_Horizontal"
 			(at 364.49 71.12 0)
 			(effects
@@
 			)
 		)
-		(property "Footprint" "Connector_PinSocket_2.54mm:PinSocket_1x03_P2.54mm_Vertical"
+		(property "Footprint" "Connector_PinSocket_2.54mm:PinSocket_1x03_P2.54mm_Horizontal"
 			(at 364.49 34.29 0)
 			(effects
@@
 	(symbol
 		(lib_id "Connector:Conn_01x03_Pin")
-		(at 430.53 71.12 0)
-		(mirror y)
+		(at 430.53 71.12 180)
 		(unit 1)
 		(exclude_from_sim no)
@@
 		(on_board yes)
 		(dnp no)
-		(fields_autoplaced yes)
 		(property "Reference" "J24"
-			(at 431.8 69.8499 0)
+			(at 431.8 72.3901 0)
 			(effects
 				(font
@@
 		)
 		(property "Value" "TM"
-			(at 431.8 72.3899 0)
+			(at 431.8 69.8501 0)
 			(effects
 				(font
@@
 			)
 		)
-		(property "Footprint" "Connector_PinHeader_2.54mm:PinHeader_1x03_P2.54mm_Vertical"
+		(property "Footprint" "Connector_PinHeader_2.54mm:PinHeader_1x03_P2.54mm_Horizontal"
 			(at 430.53 71.12 0)
 			(effects

Commit message: UPDATE: improved LVCC rail usage on MOD-XVR(4IO)
  - LVCC now powers the LEDs, the buffer driving them is powered by
    DVCC, this avoids transients caused by UI changes to propagage
    on the digital power rail
  - 74HC04 was replaced by 74HC125
  - also added decoupling capacitors to all logic chips that required
    them
  - changed footprint of Timing Module capacitor to reflect mounting
    (horizontal)
  - re-done routing and adjusted silkscreen in affected areas.
Parts:
- removed U9: 74HC04, Package_DIP:DIP-14_W7.62mm, symbol 74xx:74HC04
- added C6, C7, C8: 100nF, Capacitor_THT:C_Rect_L4.0mm_W2.5mm_P2.50mm, symbol Device:C
- added U7: 74LS125, Package_DIP:DIP-14_W7.62mm, symbol 74xx:74LS125
- C5: footprint Capacitor_THT:C_Rect_L9.0mm_W2.5mm_P7.50mm_MKT -> Capacitor_THT:CP_Radial_D5.0mm_P2.00mm
- D26: footprint LED_THT:LED_D3.0mm_Horizontal_O1.27mm_Z2.0mm -> LED_THT:LED_D3.0mm_Horizontal_O3.81mm_Z6.0mm
- D27: footprint LED_THT:LED_D3.0mm_Horizontal_O3.81mm_Z6.0mm -> LED_THT:LED_D3.0mm_Horizontal_O1.27mm_Z2.0mm
- F1, F2: value 1AF -> F1A
Connections:
- net DGND: now also C6.2, U7.1, U7.10, U7.13, U7.4, U7.7 (GND); no longer D25.1 (K), D26.1 (K), D27.1 (K), D28.1 (K)
- net DVCC: now also C6.1, U7.14 (VCC)
- net ISEC_DGND: now also U3.11, C7.2; no longer U3.10
- net ISEC_DVCC: now also C7.1
- net LVCC: now also D25.2 (A), D26.2 (A), D27.2 (A), D28.2 (A)
- net WDDM_DGND: now also C8.2
- net WDDM_DVCC: now also C8.1
- net ~{BGPIO_E_0}: now also U7.9
- net ~{BGPIO_E_1}: now also U7.12
- net ~{BGPIO_E_2}: now also U7.5
- net ~{BGPIO_E_3}: now also U7.2
- net at R32.1: now also U7.8
- net at R32.2: now also D25.1 (K); no longer D25.2 (A)
- net at R35.1: now also U7.3
- net at R35.2: now also D28.1 (K); no longer D28.2 (A)
- net at R33.1: now also U7.11
- net at R33.2: now also D26.1 (K); no longer D26.2 (A)
- net at R34.1: now also U7.6
- net at R34.2: now also D27.1 (K); no longer D27.2 (A)
- no-connect marks 18 -> 16
Other:
- moved on the sheet: D25, D26, D27, D28, R32, R33, R34, R35, U3E, U3F, U3G
